Commit message: Update MHS.urdf

File: mhs/MHS.urdf (robot description, URDF)
Before this commit: robot , 12 links, 11 joints
Links:
- added link Frame_MHS_NAVCAM
Joints:
- added joint MHS_NAVCAM: type None, parent Body_MHS_MainBody_v16, child Frame_MHS_NAVCAM, origin xyz=0.0 0.0616891 0.13743 rpy=-0.0027478 0.0580433 -1.57391594
